File: rmk-ble-keyboard.kicad_pcb (KiCad board)
At the start: 2 copper layers, 285 x 94.5 mm, 157 parts, among them J1 USB_C_Receptacle_USB2.0_16P, J2 Battery, J3 Debug, J4 RGB, J5 Reset, Q1 Si2301CDS, SW1 esc, SW10 9, SW11 0, SW12 -, SW13 =, SW14 backspace, SW15 tab, SW16 q, SW17 w, SW18 e, SW19 r, SW2 1, SW20 t, SW21 y, SW22 u, SW23 i, SW24 o, SW25 p, SW26 [, SW27 ], SW28 \, SW29 capslock, SW3 2, SW30 a, SW31 s, SW32 d, SW33 f, SW34 g, SW35 h, SW36 j, SW37 k, SW38 l, SW39 ;, SW4 3, SW40 ', SW41 enter, SW42 lshift, SW43 z, SW44 x, SW45 c, SW46 v, SW47 b, SW48 n, SW49 m, SW5 4, SW50 ,, SW51 ., SW52 /, SW53 rshift, SW54 lctrl, SW55 lgui, SW56 lalt, SW57 space, SW58 ralt, SW59 rgui, SW6 5, SW60 fn, SW61 rctrl, SW62 MSK-12C02, SW63 key, SW7 6, SW8 7, SW9 8, U2 USBLC6-2SC6, U3 TP4056, U5 AP2112K-3.3, Y1 32.768KHZ

Commit message: pcb layout
Signed-off-by: HaoboGu <haobogu@outlook.com>
Parts:
- removed J2: Battery, Connector_JST:JST_SH_SM02B-SRSS-TB_1x02-1MP_P1.00mm_Horizontal
- added J6: Battery, Connector_JST:JST_SH_SM02B-SRSS-TB_1x02-1MP_P1.00mm_Horizontal, B.Cu at (138.1, 83.5)
- added REF**: Stabilizer_Cherry_MX_2.00u, PCM_Mounting_Keyboard_Stabilizer:Stabilizer_Cherry_MX_2.00u, F.Cu at (292.9, 75.3)
- added REF**: Stabilizer_Cherry_MX_2.00u, PCM_Mounting_Keyboard_Stabilizer:Stabilizer_Cherry_MX_2.00u, F.Cu at (295.3, 38.1)
- added REF**: Stabilizer_Cherry_MX_2.00u, PCM_Mounting_Keyboard_Stabilizer:Stabilizer_Cherry_MX_2.00u, F.Cu at (50.0, 95.2)
- added REF**: Stabilizer_Cherry_MX_6.25u, PCM_Mounting_Keyboard_Stabilizer:Stabilizer_Cherry_MX_6.25u, F.Cu at (159.5, 114.3)
- added REF**: Stabilizer_Cherry_MX_2.00u, PCM_Mounting_Keyboard_Stabilizer:Stabilizer_Cherry_MX_2.00u, B.Cu at (288.1, 94.4)
- C1, C2, C3, C4, D63, R1, R2, R3, R4, R5, R6, R7, R8, R9, U2, U3, U5, Y1: moved to B.Cu
- J4: footprint Connector_PinHeader_2.54mm:PinHeader_1x03_P2.54mm_Vertical -> Connector_PinHeader_1.27mm:PinHeader_1x03_P1.27mm_Vertical
- Q1: footprint Package_TO_SOT_SMD:SOT-23-5_HandSoldering -> Package_TO_SOT_SMD:SOT-23; moved to B.Cu
- SW62: footprint MSK-12C02:SW-TH_MSK12C02 -> Button_Switch_SMD:SW_SPDT_PCM12; moved to B.Cu
- moved D64 168.7 mm to (311.5, 53.6), turned to 180 degrees
- moved U2 167.0 mm to (49.6, 47.6)
- moved R10 164.2 mm to (311.5, 55.1), turned to 180 degrees
- moved R2 162.5 mm to (38.0, 31.0), turned to 180 degrees
- moved R1 159.3 mm to (38.0, 32.5), turned to 180 degrees
- moved J5 152.8 mm to (31.0, 77.0)
- moved D62 151.2 mm to (35.3, 76.8), turned to 90 degrees
- moved J3 149.5 mm to (31.0, 65.7)
- moved R7 147.1 mm to (57.1, 31.8)
- moved J4 146.0 mm to (66.6, 31.8)
- moved SW63 119.7 mm to (290.5, 117.7), turned to -90 degrees
- moved SW62 111.7 mm to (58.7, 76.4), turned to 90 degrees
- moved R5 104.9 mm to (60.1, 83.4), turned to 90 degrees
- moved D63 73.6 mm to (100.5, 108.6), turned to 180 degrees
- moved Q1 73.0 mm to (100.6, 105.6), turned to -90 degrees
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Connections:
- U1 pad 1: /matrix/col4 -> /matrix/row1
- U1 pad 10: /matrix/row5 -> /matrix/col1
- U1 pad 2: /matrix/col3 -> /matrix/row2
- U1 pad 3: /matrix/col2 -> /matrix/row3
- U1 pad 4: /matrix/col1 -> /matrix/row4
- U1 pad 5: GND -> /matrix/row5
- U1 pad 6: /matrix/row1 -> GND
- U1 pad 7: /matrix/row2 -> /matrix/col4
- U1 pad 8: /matrix/row3 -> /matrix/col3
- U1 pad 9: /matrix/row4 -> /matrix/col2
Routing:
- net /matrix/row1: track 0.00 -> 313.0 mm, vias 0 -> 13
- net /matrix/row4: track 242.2 -> 0.00 mm
- net /matrix/col14: track 85.9 -> 99.8 mm
- net /matrix/col3: track 87.4 -> 91.0 mm
- net /matrix/col10: track 83.7 -> 87.0 mm
- net /matrix/col6: track 83.7 -> 87.0 mm
- net /matrix/col11: track 83.7 -> 87.0 mm
- net /matrix/col4: track 64.0 -> 67.0 mm
- net /matrix/col8: track 64.0 -> 67.0 mm
- net /matrix/col5: track 64.0 -> 67.0 mm
- net /matrix/col9: track 64.0 -> 67.0 mm
- net /matrix/col7: track 64.0 -> 67.0 mm
- net /matrix/col2: track 82.4 -> 85.0 mm
- net /matrix/col1: track 76.8 -> 78.9 mm
- net /matrix/col12: track 42.1 -> 44.0 mm
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
Commit message: add routes
Signed-off-by: HaoboGu <haobogu@outlook.com>
Parts:
- R5, R6, SW62: moved to F.Cu
- moved R6 96.9 mm to (36.2, 76.7), turned to 90 degrees
- moved C1 19.7 mm to (114.7, 111.0), turned to -90 degrees
- moved R3 17.8 mm to (118.4, 117.1), turned to 90 degrees
- moved C2 16.6 mm to (116.9, 117.1), turned to -90 degrees
- moved R4 15.7 mm to (115.1, 117.3), turned to 90 degrees
- moved R5 14.9 mm to (56.5, 68.9), turned to 180 degrees
- moved U3 12.7 mm to (118.3, 111.0), turned to 180 degrees
- moved Q1 6.68 mm to (100.9, 112.3), turned to 0 degrees
- moved D63 5.09 mm to (103.9, 112.4), turned to -90 degrees
- moved C4 4.14 mm to (123.2, 115.0)
- moved U5 4.14 mm to (123.5, 112.5)
- moved C3 4.14 mm to (123.2, 110.0)
- moved U2 2.89 mm to (52.4, 47.6)
- moved SW62 2.62 mm to (57.3, 74.2)
- moved D62 0.69 mm to (34.7, 76.7)
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Routing:
- net /matrix/row3: track 0.00 -> 297.1 mm, vias 0 -> 14
- net /matrix/row2: track 0.00 -> 285.0 mm, vias 0 -> 14
- net /matrix/row4: track 0.00 -> 251.3 mm, vias 0 -> 12
- net VBUS: track 0.00 -> 210.6 mm, vias 0 -> 2
- net /matrix/row5: track 47.4 -> 198.3 mm, vias 0 -> 8
- net /mcu/D+: track 0.00 -> 127.1 mm, vias 0 -> 1
- net /mcu/D-: track 0.00 -> 126.9 mm, vias 0 -> 2
- net Net-(D63--): track 0.00 -> 33.8 mm
- net /power/DP: track 0.00 -> 19.1 mm, vias 0 -> 2
- net /power/DN: track 0.00 -> 18.5 mm
- net /power/Li+: track 0.00 -> 16.4 mm
- net /power/Vin: track 0.00 -> 15.6 mm
- net Net-(J1-CC2): track 0.00 -> 12.2 mm
- net 3V3: track 0.00 -> 10.6 mm
- net Net-(J1-CC1): track 0.00 -> 9.01 mm
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Other:
- outline, holes or cut-outs redrawn

Commit message: rev 1.0
Signed-off-by: HaoboGu <haobogu@outlook.com>
Parts:
- removed SW63: key, Button_Switch_SMD:SW_Push_1P1T_XKB_TS-1187A
- J5: footprint Connector_PinHeader_2.54mm:PinHeader_1x02_P2.54mm_Vertical -> Connector_PinHeader_1.27mm:PinHeader_1x02_P1.27mm_Vertical
- moved R10 142.3 mm to (185.2, 120.8), turned to 0 degrees
- moved D64 140.1 mm to (188.6, 120.8)
- moved J5 117.6 mm to (147.1, 95.5), turned to 180 degrees
- moved R9 11.1 mm to (143.9, 83.6), turned to -90 degrees
- moved R8 9.24 mm to (142.4, 83.6), turned to 90 degrees
- moved D62 3.26 mm to (35.6, 73.6), turned to -90 degrees
- moved R6 0.63 mm to (35.6, 77.0)
Connections:
- U1 pad 12: unconnected-(U1-P0.26-Pad12) -> /mcu/caps
- U1 pad 14: unconnected-(U1-P0.06-Pad14) -> /mcu/rgb
- U1 pad 22: unconnected-(U1-P0.07-Pad22) -> /mcu/CHARGE
- U1 pad 28: /matrix/col11 -> unconnected-(U1-P15-Pad28)
- U1 pad 30: /matrix/col12 -> unconnected-(U1-P17-Pad30)
- U1 pad 32: /matrix/col13 -> unconnected-(U1-P0.20-Pad32)
- U1 pad 34: /matrix/col14 -> unconnected-(U1-P0.22-Pad34)
- U1 pad 36: Net-(U1-P1.00) -> /matrix/col11
- U1 pad 38: /mcu/rgb -> /matrix/col12
- U1 pad 40: /mcu/CHARGE -> /matrix/col13
- U1 pad 42: /mcu/caps -> /matrix/col14
Routing:
- net /matrix/row1: track 313.4 -> 519.2 mm, vias 14 -> 17
- net /matrix/row2: track 285.0 -> 468.2 mm, vias 14 -> 17
- net /matrix/row3: track 297.1 -> 464.1 mm, vias 14 -> 17
- net /matrix/col12: track 43.0 -> 200.1 mm, vias 0 -> 2
- net /matrix/row4: track 251.3 -> 401.7 mm, vias 12 -> 15
- net /matrix/col14: track 97.6 -> 245.9 mm, vias 0 -> 2
- net /mcu/rgb: track 0.00 -> 137.5 mm, vias 0 -> 4
- net /matrix/col13: track 80.2 -> 217.2 mm, vias 0 -> 2
- net /mcu/swd: track 0.00 -> 136.9 mm, vias 0 -> 1
- net /mcu/swc: track 0.00 -> 136.6 mm, vias 0 -> 2
- net 3V3: track 10.6 -> 144.4 mm, vias 0 -> 3
- net /mcu/caps: track 0.00 -> 129.2 mm, vias 0 -> 3
- net /matrix/col11: track 85.1 -> 203.2 mm, vias 0 -> 2
- net Net-(J6-Pin_1): track 0.00 -> 103.1 mm, vias 0 -> 3
- net /matrix/col1: track 77.8 -> 179.7 mm, vias 0 -> 1
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- added copper zone on B.Cu, net GND
- added copper zone on F.Cu, net GND
Other:
- outline, holes or cut-outs redrawn
- board text added: "Firmware at: github.com/haobogu/rmk"
- board text added: "rmk-ble-keyboard - v1.0 by haobogu"
- board text removed: "PCB3D_BR_TEST"
- board text removed: "PCB3D_TL_TEST"

Commit message: update production file
Signed-off-by: HaoboGu <haobogu@outlook.com>
Parts:
- J6: value Battery -> JST-SM02B-SRSS-TB
- R8: value 810K -> 820K
Routing:
- net /mcu/rgb: vias 4 -> 5
- net /mcu/charging_led: vias 3 -> 4
- net /mcu/caps: vias 3 -> 4
- net /matrix/col14: vias 2 -> 3
- net /matrix/col13: vias 2 -> 3
- net /matrix/col12: vias 2 -> 3
- net /matrix/col11: vias 2 -> 3
Changed lines of the file:
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@@
 			)
 		)
-		(property "Value" "Battery"
+		(property "Value" "JST-SM02B-SRSS-TB"
 			(at 0 -3.98 0)
 			(layer "B.Fab")
@@
 			)
 		)
-		(property "Value" "810K"
+		(property "Value" "820K"
 			(at 0 -1.43 -90)
 			(layer "B.Fab")
@@
 	)
 	(via
+		(at 130.7572 116.61115)
+		(size 0.8)
+		(drill 0.4)
+		(layers "F.Cu" "B.Cu")
+		(net 83)
+	)
+	(via
 		(at 75.81 45.085)
 		(size 0.5)
@@
 	)
 	(via
+		(at 130.7572 117.88115)
+		(size 0.8)
+		(drill 0.4)
+		(layers "F.Cu" "B.Cu")
+		(net 91)
+	)
+	(via
 		(at 41.75 86.605)
 		(size 0.8)
@@
 		(net 93)
 	)
+	(via
+		(at 130.7572 115.34115)
+		(size 0.8)
+		(drill 0.4)
+		(layers "F.Cu" "B.Cu")
+		(net 93)
+	)
 	(segment
 		(start 150.768924 123.02)
@@
 		(net 105)
 	)
+	(via
+		(at 138.0422 109.8714)
+		(size 0.8)
+		(drill 0.4)
+		(layers "F.Cu" "B.Cu")
+		(net 105)
+	)
 	(arc
 		(start 197.850762 103.99)
@@
 		(net 106)
 	)
+	(via
+		(at 139.3122 109.8714)
+		(size 0.8)
+		(drill 0.4)
+		(layers "F.Cu" "B.Cu")
+		(net 106)
+	)
 	(arc
 		(start 198.319046 104.58)
@@
 		(net 107)
 	)
+	(via
+		(at 140.5822 109.8714)
+		(size 0.8)
+		(drill 0.4)
+		(layers "F.Cu" "B.Cu")
+		(net 107)
+	)
 	(arc
 		(start 198.714429 105.17)
@@
 		(layers "F.Cu" "B.Cu")
 		(net 108)
+	)
+	(via
+		(at 141.8472 109.8714)
+		(size 0.8)
+		(drill 0.4)
+		(layers "F.Cu" "B.Cu")
+		(net 108)

Commit message: feat: update rev 1
Signed-off-by: HaoboGu <haobogu@outlook.com>
Parts:
- added ?: , , F.Cu at (138.0, 109.9)
- added ?: , , F.Cu at (130.8, 110.3)
- added ?: , , F.Cu at (141.8, 109.9)
- added ?: , , F.Cu at (139.3, 109.9)
- added ?: , , F.Cu at (130.8, 117.9)
- added ?: , , F.Cu at (130.8, 115.3)
- added ?: , , F.Cu at (140.6, 109.9)
- added ?: , , F.Cu at (130.8, 114.1)
- added ?: , , F.Cu at (130.8, 111.5)
- added ?: , , F.Cu at (130.8, 116.6)
- added ?: , , F.Cu at (128.5, 112.2)
Routing:
- net GND: vias 100 -> 98
- net /mcu/rgb: vias 5 -> 4
- net /mcu/charging_led: vias 4 -> 3
- net /mcu/caps: vias 4 -> 3
- net /mcu/bat_adc: vias 2 -> 1
- net /mcu/CHARGE: vias 4 -> 3
- net /matrix/col14: vias 3 -> 2
- net /matrix/col13: vias 3 -> 2
- net /matrix/col12: vias 3 -> 2
- net /matrix/col11: vias 3 -> 2
